Commit message: 描述文件修改

File: src/dual_fr3_description/urdf/dual_fr3.urdf.xacro (robot description, xacro)
@@ -4,5 +4,7 @@
   <xacro:include filename="$(find franka_description)/robots/common/franka_robot.xacro"/>
   <xacro:property name="joint_limits" value="${xacro.load_yaml('$(find franka_description)/robots/fr3/joint_limits.yaml')}" />
-  <xacro:property name="connected_to" value="base_link" />
+  <xacro:property name="kinematics" value="${xacro.load_yaml('$(find franka_description)/robots/fr3/kinematics.yaml')}" />
+  <xacro:property name="inertials" value="${xacro.load_yaml('$(find franka_description)/robots/fr3/inertials.yaml')}" />
+  <xacro:property name="dynamics" value="${xacro.load_yaml('$(find franka_description)/robots/fr3/dynamics.yaml')}" />
   <xacro:mr1000_description_macro/>
   <link name="world"/>
@@ -12,17 +14,31 @@
     <origin xyz="0 0 0" rpy="0 0 0"/>
   </joint>
-  <xacro:franka_robot arm_id="left"
-                      connected_to="${connected_to}"
-                      xyz="0 0.3 0.5"
-                      rpy="0 0 0"
+  <xacro:franka_robot arm_id="fr3"
+                      arm_prefix="left_"
+                      connected_to=""
                       safety_distance="0.03"
                       gazebo="false"
-                      joint_limits="${joint_limits}"/>
-  <xacro:franka_robot arm_id="right"
-                      connected_to="${connected_to}"
-                      xyz="0 -0.3 0.5"
-                      rpy="0 0 0"
+                      joint_limits="${joint_limits}"
+                      kinematics="${kinematics}"
+                      inertials="${inertials}"
+                      dynamics="${dynamics}"/>
+  <joint name="left_fr3_mount_joint" type="fixed">
+      <parent link="base_link" />
+      <child link="left_fr3_link0" />
+      <origin xyz="0.153 0.06 0.9685" rpy="-1.5707963267949 -1.5707963267949 0" />
+  </joint>
+  <xacro:franka_robot arm_id="fr3"
+                      arm_prefix="right_"
+                      connected_to=""
                       safety_distance="0.03"
                       gazebo="false"
-                      joint_limits="${joint_limits}"/>
+                      joint_limits="${joint_limits}"
+                      kinematics="${kinematics}"
+                      inertials="${inertials}"
+                      dynamics="${dynamics}"/>
+  <joint name="right_fr3_mount_joint" type="fixed">
+      <parent link="base_link" />
+      <child link="right_fr3_link0" />
+      <origin xyz="0.153 -0.06 0.9685" rpy="1.5707963267949 -1.5707963267949 0" />
+  </joint>
 </robot>

File: src/dual_fr3_description/urdf/mr1000_macro.xacro (robot description, xacro)
@@ -26,20 +26,27 @@
         rpy="0 0 0" />
       <geometry>
+        <!-- <mesh
+          filename="package://dual_fr3_description/meshes/base_link.STL" /> -->
+        <box size="0.8 0.6 0.3" />
+      </geometry>
+      <material
+        name="">
+        <color
+          rgba="0.752941176470588 0.752941176470588 0.752941176470588 1" />
+      </material>
+    </visual>
+    <!-- <collision>
+      <origin
+        xyz="0 0 0"
+        rpy="0 0 0" />
+      <geometry>
         <mesh
           filename="package://dual_fr3_description/meshes/base_link.STL" />
       </geometry>
-      <material
-        name="">
-        <color
-          rgba="0.752941176470588 0.752941176470588 0.752941176470588 1" />
-      </material>
-    </visual>
-    <collision>
-      <origin
-        xyz="0 0 0"
-        rpy="0 0 0" />
-      <geometry>
-        <mesh
-          filename="package://dual_fr3_description/meshes/base_link.STL" />
+    </collision> -->
+    <collision>
+      <origin xyz="0 0 0" rpy="0 0 0" />
+      <geometry>
+        <box size="0.8 0.6 0.3" />
       </geometry>
     </collision>
@@ -66,20 +73,27 @@
         rpy="0 0 0" />
       <geometry>
-        <mesh
-          filename="package://dual_fr3_description/meshes/wheel_LF_link.STL" />
-      </geometry>
-      <material
-        name="">
-        <color
-          rgba="1 0.945098039215686 0.905882352941176 1" />
-      </material>
-    </visual>
-    <collision>
-      <origin
-        xyz="0 0 0"
-        rpy="0 0 0" />
-      <geometry>
-        <mesh
-          filename="package://dual_fr3_description/meshes/wheel_LF_link.STL" />
+        <!-- <mesh
+          filename="package://dual_fr3_description/meshes/wheel_LF_link.STL" /> -->
+        <cylinder radius="0.1" length="0.05"/>
+      </geometry>
+      <material
+        name="">
+        <color
+          rgba="1 0.945098039215686 0.905882352941176 1" />
+      </material>
+    </visual>
+    <!-- <collision>
+      <origin
+        xyz="0 0 0"
+        rpy="0 0 0" />
+      <geometry>
+        <mesh
+          filename="package://dual_fr3_description/meshes/wheel_LF_link.STL" />
+      </geometry>
+    </collision> -->
+    <collision>
+      <origin xyz="0 0 0" rpy="${pi/2} 0 0" />
+      <geometry>
+        <cylinder radius="0.1" length="0.05"/>
       </geometry>
     </collision>
@@ -119,20 +133,27 @@
         rpy="0 0 0" />
       <geometry>
-        <mesh
-          filename="package://dual_fr3_description/meshes/wheel_LF_link.STL" />
-      </geometry>
-      <material
-        name="">
-        <color
-          rgba="1 0.945098039215686 0.905882352941176 1" />
-      </material>
-    </visual>
-    <collision>
-      <origin
-        xyz="0 0 0"
-        rpy="0 0 0" />
-      <geometry>
-        <mesh
-          filename="package://dual_fr3_description/meshes/wheel_LF_link.STL" />
+        <!-- <mesh
+          filename="package://dual_fr3_description/meshes/wheel_LF_link.STL" /> -->
+        <cylinder radius="0.1" length="0.05"/>
+      </geometry>
+      <material
+        name="">
+        <color
+          rgba="1 0.945098039215686 0.905882352941176 1" />
+      </material>
+    </visual>
+    <!-- <collision>
+      <origin
+        xyz="0 0 0"
+        rpy="0 0 0" />
+      <geometry>
+        <mesh
+          filename="package://dual_fr3_description/meshes/wheel_LF_link.STL" />
+      </geometry>
+    </collision> -->
+    <collision>
+      <origin xyz="0 0 0" rpy="${pi/2} 0 0" />
+      <geometry>
+        <cylinder radius="0.1" length="0.05"/>
       </geometry>
     </collision>
@@ -172,20 +193,27 @@
         rpy="0 0 0" />
       <geometry>
-        <mesh
-          filename="package://dual_fr3_description/meshes/wheel_LF_link.STL" />
-      </geometry>
-      <material
-        name="">
-        <color
-          rgba="1 0.945098039215686 0.905882352941176 1" />
-      </material>
-    </visual>
-    <collision>
-      <origin
-        xyz="0 0 0"
-        rpy="0 0 0" />
-      <geometry>
-        <mesh
-          filename="package://dual_fr3_description/meshes/wheel_LF_link.STL" />
+        <!-- <mesh
+          filename="package://dual_fr3_description/meshes/wheel_LF_link.STL" /> -->
+        <cylinder radius="0.1" length="0.05"/>
+      </geometry>
+      <material
+        name="">
+        <color
+          rgba="1 0.945098039215686 0.905882352941176 1" />
+      </material>
+    </visual>
+    <!-- <collision>
+      <origin
+        xyz="0 0 0"
+        rpy="0 0 0" />
+      <geometry>
+        <mesh
+          filename="package://dual_fr3_description/meshes/wheel_LF_link.STL" />
+      </geometry>
+    </collision> -->
+    <collision>
+      <origin xyz="0 0 0" rpy="${pi/2} 0 0" />
+      <geometry>
+        <cylinder radius="0.1" length="0.05"/>
       </geometry>
     </collision>
@@ -225,20 +253,27 @@
         rpy="0 0 0" />
       <geometry>
-        <mesh
-          filename="package://dual_fr3_description/meshes/wheel_LF_link.STL" />
-      </geometry>
-      <material
-        name="">
-        <color
-          rgba="1 0.945098039215686 0.905882352941176 1" />
-      </material>
-    </visual>
-    <collision>
-      <origin
-        xyz="0 0 0"
-        rpy="0 0 0" />
-      <geometry>
-        <mesh
-          filename="package://dual_fr3_description/meshes/wheel_LF_link.STL" />
+        <!-- <mesh
+          filename="package://dual_fr3_description/meshes/wheel_LF_link.STL" /> -->
+        <cylinder radius="0.1" length="0.05"/>
+      </geometry>
+      <material
+        name="">
+        <color
+          rgba="1 0.945098039215686 0.905882352941176 1" />
+      </material>
+    </visual>
+    <!-- <collision>
+      <origin
+        xyz="0 0 0"
+        rpy="0 0 0" />
+      <geometry>
+        <mesh
+          filename="package://dual_fr3_description/meshes/wheel_LF_link.STL" />
+      </geometry>
+    </collision> -->
+    <collision>
+      <origin xyz="0 0 0" rpy="${pi/2} 0 0" />
+      <geometry>
+        <cylinder radius="0.1" length="0.05"/>
       </geometry>
     </collision>

Commit message: 模型URDF文件提交

File: src/dual_fr3_description/urdf/dual_fr3.urdf.xacro (robot description, xacro)
@@ -1,11 +1,4 @@
 <?xml version="1.0"?>
 <robot xmlns:xacro="http://www.ros.org/wiki/xacro" name="dual_fr3_robot">
-  <xacro:include filename="$(find dual_fr3_description)/urdf/mr1000_macro.xacro"/>
-  <xacro:include filename="$(find franka_description)/robots/common/franka_robot.xacro"/>
-  <xacro:property name="joint_limits" value="${xacro.load_yaml('$(find franka_description)/robots/fr3/joint_limits.yaml')}" />
-  <xacro:property name="kinematics" value="${xacro.load_yaml('$(find franka_description)/robots/fr3/kinematics.yaml')}" />
-  <xacro:property name="inertials" value="${xacro.load_yaml('$(find franka_description)/robots/fr3/inertials.yaml')}" />
-  <xacro:property name="dynamics" value="${xacro.load_yaml('$(find franka_description)/robots/fr3/dynamics.yaml')}" />
-  <xacro:mr1000_description_macro/>
   <link name="world"/>
   <joint name="world_to_base" type="fixed">
@@ -14,4 +7,22 @@
     <origin xyz="0 0 0" rpy="0 0 0"/>
   </joint>
+  <xacro:include filename="$(find dual_fr3_description)/urdf/mr1000_macro.xacro"/>
+  <joint name="left_fr3_fixed_joint" type="fixed">
+      <parent link="base_link" />
+      <child link="left_fr3_link0" />
+      <origin xyz="0.153 0.06 0.9685" rpy="-1.5707963267949 -1.5707963267949 0" />
+  </joint>
+  <joint name="right_fr3_fixed_joint" type="fixed">
+      <parent link="base_link" />
+      <child link="right_fr3_link0" />
+      <origin xyz="0.153 -0.06 0.9685" rpy="1.5707963267949 -1.5707963267949 0" />
+  </joint>
+  <xacro:include filename="$(find franka_description)/robots/common/franka_robot.xacro"/>
+  <!-- 加载 YAML 配置 -->
+  <xacro:property name="joint_limits" value="${xacro.load_yaml('$(find franka_description)/robots/fr3/joint_limits.yaml')}" />
+  <xacro:property name="kinematics" value="${xacro.load_yaml('$(find franka_description)/robots/fr3/kinematics.yaml')}" />
+  <xacro:property name="inertials" value="${xacro.load_yaml('$(find franka_description)/robots/fr3/inertials.yaml')}" />
+  <xacro:property name="dynamics" value="${xacro.load_yaml('$(find franka_description)/robots/fr3/dynamics.yaml')}" />
+  <xacro:property name="accelerometer_config" value="${xacro.load_yaml('$(find franka_description)/robots/fr3/accelerometers.yaml')}" />
   <xacro:franka_robot arm_id="fr3"
                       arm_prefix="left_"
@@ -23,9 +34,4 @@
                       inertials="${inertials}"
                       dynamics="${dynamics}"/>
-  <joint name="left_fr3_mount_joint" type="fixed">
-      <parent link="base_link" />
-      <child link="left_fr3_link0" />
-      <origin xyz="0.153 0.06 0.9685" rpy="-1.5707963267949 -1.5707963267949 0" />
-  </joint>
   <xacro:franka_robot arm_id="fr3"
                       arm_prefix="right_"
@@ -37,8 +43,3 @@
                       inertials="${inertials}"
                       dynamics="${dynamics}"/>
-  <joint name="right_fr3_mount_joint" type="fixed">
-      <parent link="base_link" />
-      <child link="right_fr3_link0" />
-      <origin xyz="0.153 -0.06 0.9685" rpy="1.5707963267949 -1.5707963267949 0" />
-  </joint>
 </robot>

File: src/dual_fr3_description/urdf/mr1000_macro.xacro (robot description, xacro)
@@ -26,7 +26,6 @@
         rpy="0 0 0" />
       <geometry>
-        <!-- <mesh
-          filename="package://dual_fr3_description/meshes/base_link.STL" /> -->
-        <box size="0.8 0.6 0.3" />
+        <mesh
+          filename="package://dual_fr3_description/meshes/base_link.STL" />
       </geometry>
       <material
@@ -73,7 +72,6 @@
         rpy="0 0 0" />
       <geometry>
-        <!-- <mesh
-          filename="package://dual_fr3_description/meshes/wheel_LF_link.STL" /> -->
-        <cylinder radius="0.1" length="0.05"/>
+        <mesh
+          filename="package://dual_fr3_description/meshes/wheel_LF_link.STL" />
       </geometry>
       <material
@@ -133,21 +131,20 @@
         rpy="0 0 0" />
       <geometry>
-        <!-- <mesh
-          filename="package://dual_fr3_description/meshes/wheel_LF_link.STL" /> -->
-        <cylinder radius="0.1" length="0.05"/>
-      </geometry>
-      <material
-        name="">
-        <color
-          rgba="1 0.945098039215686 0.905882352941176 1" />
-      </material>
-    </visual>
-    <!-- <collision>
-      <origin
-        xyz="0 0 0"
-        rpy="0 0 0" />
-      <geometry>
-        <mesh
-          filename="package://dual_fr3_description/meshes/wheel_LF_link.STL" />
+        <mesh
+          filename="package://dual_fr3_description/meshes/wheel_LB_link.STL" />
+      </geometry>
+      <material
+        name="">
+        <color
+          rgba="1 0.945098039215686 0.905882352941176 1" />
+      </material>
+    </visual>
+    <!-- <collision>
+      <origin
+        xyz="0 0 0"
+        rpy="0 0 0" />
+      <geometry>
+        <mesh
+          filename="package://dual_fr3_description/meshes/wheel_LB_link.STL" />
       </geometry>
     </collision> -->
@@ -193,21 +190,20 @@
         rpy="0 0 0" />
       <geometry>
-        <!-- <mesh
-          filename="package://dual_fr3_description/meshes/wheel_LF_link.STL" /> -->
-        <cylinder radius="0.1" length="0.05"/>
-      </geometry>
-      <material
-        name="">
-        <color
-          rgba="1 0.945098039215686 0.905882352941176 1" />
-      </material>
-    </visual>
-    <!-- <collision>
-      <origin
-        xyz="0 0 0"
-        rpy="0 0 0" />
-      <geometry>
-        <mesh
-          filename="package://dual_fr3_description/meshes/wheel_LF_link.STL" />
+        <mesh
+          filename="package://dual_fr3_description/meshes/wheel_RF_link.STL" />
+      </geometry>
+      <material
+        name="">
+        <color
+          rgba="1 0.945098039215686 0.905882352941176 1" />
+      </material>
+    </visual>
+    <!-- <collision>
+      <origin
+        xyz="0 0 0"
+        rpy="0 0 0" />
+      <geometry>
+        <mesh
+          filename="package://dual_fr3_description/meshes/wheel_RF_link.STL" />
       </geometry>
     </collision> -->
@@ -253,21 +249,20 @@
         rpy="0 0 0" />
       <geometry>
-        <!-- <mesh
-          filename="package://dual_fr3_description/meshes/wheel_LF_link.STL" /> -->
-        <cylinder radius="0.1" length="0.05"/>
-      </geometry>
-      <material
-        name="">
-        <color
-          rgba="1 0.945098039215686 0.905882352941176 1" />
-      </material>
-    </visual>
-    <!-- <collision>
-      <origin
-        xyz="0 0 0"
-        rpy="0 0 0" />
-      <geometry>
-        <mesh
-          filename="package://dual_fr3_description/meshes/wheel_LF_link.STL" />
+        <mesh
+          filename="package://dual_fr3_description/meshes/wheel_RB_link.STL" />
+      </geometry>
+      <material
+        name="">
+        <color
+          rgba="1 0.945098039215686 0.905882352941176 1" />
+      </material>
+    </visual>
+    <!-- <collision>
+      <origin
+        xyz="0 0 0"
+        rpy="0 0 0" />
+      <geometry>
+        <mesh
+          filename="package://dual_fr3_description/meshes/wheel_RB_link.STL" />
       </geometry>
     </collision> -->
