Commit message: franka双臂复合机器人仿真环境功能包提交

File: src/dual_fr3_description/urdf/dual_fr3.urdf.xacro (robot description, xacro)
@@ -1,4 +1,9 @@
 <?xml version="1.0"?>
 <robot xmlns:xacro="http://www.ros.org/wiki/xacro" name="dual_fr3_robot">
+  <xacro:include filename="$(find dual_fr3_description)/urdf/mr1000_macro.xacro"/>
+  <xacro:include filename="$(find franka_description)/robots/common/franka_arm.xacro" />
+  <xacro:include filename="$(find franka_description)/end_effectors/common/franka_hand.xacro" />
+  <xacro:include filename="$(find franka_description)/end_effectors/common/utils.xacro" />
+  <!-- 基座链接 -->
   <link name="world"/>
   <joint name="world_to_base" type="fixed">
@@ -7,39 +12,68 @@
     <origin xyz="0 0 0" rpy="0 0 0"/>
   </joint>
-  <xacro:include filename="$(find dual_fr3_description)/urdf/mr1000_macro.xacro"/>
-  <joint name="left_fr3_fixed_joint" type="fixed">
+  <xacro:mr1000_description_macro />
+  <xacro:arg name="arm_id" default="fr3" />
+  <xacro:arg name="left_arm_prefix" default="left_" />
+  <xacro:arg name="right_arm_prefix" default="right_" />
+  <!-- 手动创建两个franka连接到base_link的joint，防止franka的urdf自动创建parent link -->
+  <joint name="$(arg left_arm_prefix)$(arg arm_id)_fixed_joint" type="fixed">
       <parent link="base_link" />
-      <child link="left_fr3_link0" />
+      <child link="$(arg left_arm_prefix)$(arg arm_id)_link0" />
       <origin xyz="0.153 0.06 0.9685" rpy="-1.5707963267949 -1.5707963267949 0" />
   </joint>
-  <joint name="right_fr3_fixed_joint" type="fixed">
+  <joint name="$(arg right_arm_prefix)$(arg arm_id)_fixed_joint" type="fixed">
       <parent link="base_link" />
-      <child link="right_fr3_link0" />
+      <child link="$(arg right_arm_prefix)$(arg arm_id)_link0" />
       <origin xyz="0.153 -0.06 0.9685" rpy="1.5707963267949 -1.5707963267949 0" />
   </joint>
-  <xacro:include filename="$(find franka_description)/robots/common/franka_robot.xacro"/>
-  <!-- 加载 YAML 配置 -->
-  <xacro:property name="joint_limits" value="${xacro.load_yaml('$(find franka_description)/robots/fr3/joint_limits.yaml')}" />
-  <xacro:property name="kinematics" value="${xacro.load_yaml('$(find franka_description)/robots/fr3/kinematics.yaml')}" />
-  <xacro:property name="inertials" value="${xacro.load_yaml('$(find franka_description)/robots/fr3/inertials.yaml')}" />
-  <xacro:property name="dynamics" value="${xacro.load_yaml('$(find franka_description)/robots/fr3/dynamics.yaml')}" />
-  <xacro:property name="accelerometer_config" value="${xacro.load_yaml('$(find franka_description)/robots/fr3/accelerometers.yaml')}" />
-  <xacro:franka_robot arm_id="fr3"
-                      arm_prefix="left_"
-                      connected_to=""
-                      safety_distance="0.03"
-                      gazebo="false"
-                      joint_limits="${joint_limits}"
-                      kinematics="${kinematics}"
-                      inertials="${inertials}"
-                      dynamics="${dynamics}"/>
-  <xacro:franka_robot arm_id="fr3"
-                      arm_prefix="right_"
-                      connected_to=""
-                      safety_distance="0.03"
-                      gazebo="false"
-                      joint_limits="${joint_limits}"
-                      kinematics="${kinematics}"
-                      inertials="${inertials}"
-                      dynamics="${dynamics}"/>
+  <!-- 左臂 -->
+  <xacro:franka_arm
+      arm_id="$(arg arm_id)"
+      arm_prefix="$(arg left_arm_prefix)"
+      joint_limits="${xacro.load_yaml('$(find franka_description)/robots/$(arg arm_id)/joint_limits.yaml')}"
+      inertials="${xacro.load_yaml('$(find franka_description)/robots/$(arg arm_id)/inertials.yaml')}"
+      kinematics="${xacro.load_yaml('$(find franka_description)/robots/$(arg arm_id)/kinematics.yaml')}"
+      dynamics="${xacro.load_yaml('$(find franka_description)/robots/$(arg arm_id)/dynamics.yaml')}"
+      accelerometer_config="${xacro.load_yaml('$(find franka_description)/robots/$(arg arm_id)/accelerometers.yaml')}"
+      connected_to=""
+      xyz='0.153 0.06 0.9685'
+      rpy='-1.5707963267949 -1.5707963267949 0'
+      gazebo="false">
+  </xacro:franka_arm>
+  <!-- 右臂 -->
+  <xacro:franka_arm
+      arm_id="$(arg arm_id)"
+      arm_prefix="$(arg right_arm_prefix)"
+      joint_limits="${xacro.load_yaml('$(find franka_description)/robots/$(arg arm_id)/joint_limits.yaml')}"
+      inertials="${xacro.load_yaml('$(find franka_description)/robots/$(arg arm_id)/inertials.yaml')}"
+      kinematics="${xacro.load_yaml('$(find franka_description)/robots/$(arg arm_id)/kinematics.yaml')}"
+      dynamics="${xacro.load_yaml('$(find franka_description)/robots/$(arg arm_id)/dynamics.yaml')}"
+      accelerometer_config="${xacro.load_yaml('$(find franka_description)/robots/$(arg arm_id)/accelerometers.yaml')}"
+      connected_to=""
+      xyz='0.153 -0.06 0.9685'
+      rpy='1.5707963267949 -1.5707963267949 0'
+      gazebo="false">
+  </xacro:franka_arm>
+  <!-- 左手 -->
+  <xacro:franka_hand
+    arm_id="$(arg arm_id)"
+    arm_prefix="$(arg left_arm_prefix)"
+    connected_to="$(arg left_arm_prefix)$(arg arm_id)_link8"
+    ee_id="franka_hand_white"
+    ee_inertials="${xacro.load_yaml('$(find franka_description)/end_effectors/franka_hand/inertials.yaml')}"
+    xyz_ee='0 0 0.002'
+    rpy_ee='0 0 -0.785398163'
+    gazebo="false">
+  </xacro:franka_hand>
+  <!-- 右手 -->
+  <xacro:franka_hand
+    arm_id="$(arg arm_id)"
+    arm_prefix="$(arg right_arm_prefix)"
+    connected_to="$(arg right_arm_prefix)$(arg arm_id)_link8"
+    ee_id="franka_hand_white"
+    ee_inertials="${xacro.load_yaml('$(find franka_description)/end_effectors/franka_hand/inertials.yaml')}"
+    xyz_ee='0 0 0.002'
+    rpy_ee='0 0 -0.785398163'
+    gazebo="false">
+  </xacro:franka_hand>
 </robot>

File: src/dual_fr3_description/urdf/mr1000_macro.xacro (robot description, xacro)
@@ -35,5 +35,5 @@
       </material>
     </visual>
-    <!-- <collision>
+    <collision>
       <origin
         xyz="0 0 0"
@@ -42,10 +42,4 @@
         <mesh
           filename="package://dual_fr3_description/meshes/base_link.STL" />
-      </geometry>
-    </collision> -->
-    <collision>
-      <origin xyz="0 0 0" rpy="0 0 0" />
-      <geometry>
-        <box size="0.8 0.6 0.3" />
       </geometry>
     </collision>
@@ -81,5 +75,5 @@
       </material>
     </visual>
-    <!-- <collision>
+    <collision>
       <origin
         xyz="0 0 0"
@@ -89,15 +83,9 @@
           filename="package://dual_fr3_description/meshes/wheel_LF_link.STL" />
       </geometry>
-    </collision> -->
-    <collision>
-      <origin xyz="0 0 0" rpy="${pi/2} 0 0" />
-      <geometry>
-        <cylinder radius="0.1" length="0.05"/>
-      </geometry>
     </collision>
   </link>
   <joint
     name="wheel_LF_joint"
-    type="continuous">
+    type="fixed">
     <origin
       xyz="0.212 0.323100000000001 0"
@@ -140,5 +128,5 @@
       </material>
     </visual>
-    <!-- <collision>
+    <collision>
       <origin
         xyz="0 0 0"
@@ -148,15 +136,9 @@
           filename="package://dual_fr3_description/meshes/wheel_LB_link.STL" />
       </geometry>
-    </collision> -->
-    <collision>
-      <origin xyz="0 0 0" rpy="${pi/2} 0 0" />
-      <geometry>
-        <cylinder radius="0.1" length="0.05"/>
-      </geometry>
     </collision>
   </link>
   <joint
     name="wheel_LB_joint"
-    type="continuous">
+    type="fixed">
     <origin
       xyz="-0.212 0.323099999999999 0"
@@ -199,5 +181,5 @@
       </material>
     </visual>
-    <!-- <collision>
+    <collision>
       <origin
         xyz="0 0 0"
@@ -207,15 +189,9 @@
           filename="package://dual_fr3_description/meshes/wheel_RF_link.STL" />
       </geometry>
-    </collision> -->
-    <collision>
-      <origin xyz="0 0 0" rpy="${pi/2} 0 0" />
-      <geometry>
-        <cylinder radius="0.1" length="0.05"/>
-      </geometry>
     </collision>
   </link>
   <joint
     name="wheel_RF_joint"
-    type="continuous">
+    type="fixed">
     <origin
       xyz="0.212000000000003 -0.3231 0"
@@ -258,5 +234,5 @@
       </material>
     </visual>
-    <!-- <collision>
+    <collision>
       <origin
         xyz="0 0 0"
@@ -266,15 +242,9 @@
           filename="package://dual_fr3_description/meshes/wheel_RB_link.STL" />
       </geometry>
-    </collision> -->
-    <collision>
-      <origin xyz="0 0 0" rpy="${pi/2} 0 0" />
-      <geometry>
-        <cylinder radius="0.1" length="0.05"/>
-      </geometry>
     </collision>
   </link>
   <joint
     name="wheel_RB_joint"
-    type="continuous">
+    type="fixed">
     <origin
       xyz="-0.211999999999997 -0.323100000000002 0"

File: src/dual_fr3_description/urdf/robot.urdf (robot description, URDF)
Before this commit: robot robot, 30 links, 29 joints
Links:
- removed link mk1000_fr3_link0_accelerometer_bottom
- removed link mk1000_fr3_link0_accelerometer_top
- removed link mk1000_fr3_link1_accelerometer_bottom
- removed link mk1000_fr3_link1_accelerometer_top
- removed link mk1000_fr3_link2_accelerometer_bottom
- removed link mk1000_fr3_link2_accelerometer_top
- removed link mk1000_fr3_link3_accelerometer_bottom
- removed link mk1000_fr3_link3_accelerometer_top
- removed link mk1000_fr3_link4_accelerometer_bottom
- removed link mk1000_fr3_link4_accelerometer_top
- removed link mk1000_fr3_link5_accelerometer_bottom
- removed link mk1000_fr3_link5_accelerometer_top
- link base_link: geometry collision mesh filename=package://dual_fr3_description/meshes/base_link.STL; visual mesh filename=package://dual_fr3_description/meshes/base_link.STL
- link mk1000_fr3_hand_tcp: mass None -> 0.001; geometry collision sphere radius=0.001; visual sphere radius=0.001
- link mk1000_fr3_link8: mass None -> 0.001; geometry collision sphere radius=0.001; visual sphere radius=0.001
- link wheel_LB_link: geometry collision mesh filename=package://dual_fr3_description/meshes/wheel_LB_link.STL; visual mesh filename=package://dual_fr3_description/meshes/wheel_LB_link.STL
- link wheel_LF_LINK: geometry collision mesh filename=package://dual_fr3_description/meshes/wheel_LF_link.STL; visual mesh filename=package://dual_fr3_description/meshes/wheel_LF_link.STL
- link wheel_RB_link: geometry collision mesh filename=package://dual_fr3_description/meshes/wheel_RB_link.STL; visual mesh filename=package://dual_fr3_description/meshes/wheel_RB_link.STL
- link wheel_RF_link: geometry collision mesh filename=package://dual_fr3_description/meshes/wheel_RF_link.STL; visual mesh filename=package://dual_fr3_description/meshes/wheel_RF_link.STL
Joints:
- removed joint mk1000_fr3_link0_accelerometer_bottom_joint
- removed joint mk1000_fr3_link0_accelerometer_top_joint
- removed joint mk1000_fr3_link1_accelerometer_bottom_joint
- removed joint mk1000_fr3_link1_accelerometer_top_joint
- removed joint mk1000_fr3_link2_accelerometer_bottom_joint
- removed joint mk1000_fr3_link2_accelerometer_top_joint
- removed joint mk1000_fr3_link3_accelerometer_bottom_joint
- removed joint mk1000_fr3_link3_accelerometer_top_joint
- removed joint mk1000_fr3_link4_accelerometer_bottom_joint
- removed joint mk1000_fr3_link4_accelerometer_top_joint
- removed joint mk1000_fr3_link5_accelerometer_bottom_joint
- removed joint mk1000_fr3_link5_accelerometer_top_joint
